Commit message: Started Applying skid drive controller

File: project_ws/urdf/vehicle.urdf (robot description, URDF)
Before this commit: robot vehicle, 5 links, 4 joints
Links:
- added link camera_link, mass 0.4; collision box size=0.1 0.1 0.1; visual box size=0.05 0.05 0.05
Joints:
- added joint joint_base_to_camera_link: type fixed, parent base_link, child camera_link, origin xyz=0.05 0.21 0.155

File: project_ws/urdf/vehiclediffdrive.urdf (robot description, URDF)
Before this commit: robot vehiclediffdrive, 5 links, 4 joints
Links:
- added link camera_link, mass 0.4; collision box size=0.1 0.1 0.1; visual box size=0.05 0.05 0.05
Joints:
- added joint joint_base_to_camera_link: type fixed, parent base_link, child camera_link, origin xyz=0.05 0.21 0.155
