Commit message: Applying skid driver controller

File: project_ws/urdf/vehiclediffdrive.urdf (robot description, URDF)
Before this commit: robot vehiclediffdrive, 6 links, 5 joints
Links:
- link base_link: geometry collision box size=0.2 0.4 0.1; visual box size=0.2 0.4 0.1
- link camera_link: geometry collision box size=0.05 0.05 0.05; visual box size=0.05 0.05 0.05
- link left_back_wheel: mass 1 -> 0.5
- link left_front_wheel: mass 1 -> 0.5
- link right_back_wheel: mass 1 -> 0.5
- link right_front_wheel: mass 1 -> 0.5
Joints:
- joint joint_base_to_camera_link: origin xyz=0.05 0.21 0.155 -> xyz=0.05 0.14 0.165
- joint joint_base_to_left_back_wheel: origin xyz=0.165 -0.24 0.015 rpy=1.57 1.57 1.57 -> xyz=-0.115 -0.09 0.07 rpy=1.57079633 1.57079633 1.57079633
- joint joint_base_to_left_front_wheel: origin xyz=-0.165 0.24 0.015 rpy=1.57 1.57 1.57 -> xyz=-0.115 0.09 0.07 rpy=1.57079633 1.57079633 1.57079633
- joint joint_base_to_right_back_wheel: origin xyz=-0.165 -0.24 0.015 rpy=1.57 1.57 1.57 -> xyz=0.115 -0.09 0.07 rpy=1.57079633 1.57079633 1.57079633
- joint joint_base_to_right_front_wheel: origin xyz=0.165 0.24 0.015 rpy=1.57 1.57 1.57 -> xyz=0.115 0.09 0.07 rpy=1.57079633 1.57079633 1.57079633

Commit message: Rostopic cmd velocity working established

File: project_ws/urdf/vehiclediffdrive.urdf (robot description, URDF)
Before this commit: robot vehiclediffdrive, 6 links, 5 joints
Links:
- link base_link: mass 1 -> 21.6
- link left_back_wheel: mass 0.5 -> 0.54
- link left_front_wheel: mass 0.5 -> 0.54
- link right_back_wheel: mass 0.5 -> 0.54
- link right_front_wheel: mass 0.5 -> 0.54
Joints:
- joint joint_base_to_left_back_wheel: axis (none) -> 0 0 1
- joint joint_base_to_left_front_wheel: axis (none) -> 0 0 1
- joint joint_base_to_right_back_wheel: axis (none) -> 0 0 1
- joint joint_base_to_right_front_wheel: axis (none) -> 0 0 1

Commit message: Initial phase completed

File: project_ws/urdf/vehiclediffdrive.urdf (robot description, URDF)
Before this commit: robot vehiclediffdrive, 6 links, 5 joints
Joints:
- joint joint_base_to_camera_link: origin xyz=0.05 0.14 0.165 -> xyz=0.05 -0.14 0.165 rpy=0 0 4.712 

Commit message: Laser sensor added

File: project_ws/urdf/vehiclediffdrive.urdf (robot description, URDF)
Before this commit: robot vehiclediffdrive, 6 links, 5 joints
Links:
- added link laser_link, mass 0.4; collision box size=0.05 0.05 0.08; visual box size=0.05 0.05 0.08
- link camera_link: geometry collision box size=0.05 0.05 0.08; visual box size=0.05 0.05 0.08
Joints:
- added joint joint_base_to_laser_link: type fixed, parent base_link, child laser_link, origin xyz=-0.04 -0.14 0.165 rpy=0 0 4.712 
